File: Schematics/SolarChargerV2.kicad_sch (KiCad schematic)
At the start: 20 parts

Commit message: updates and changes
Parts:
- BT1: renamed from BT?; value (none) -> Battery_Cell
- C1: renamed from C?; value (none) -> 10u
- C2: renamed from C?; value (none) -> 100n
- C3: renamed from C?; value (none) -> 82n
- C4: renamed from C?; value (none) -> 195p
- C5: renamed from C?; value (none) -> 1n
- C6: renamed from C?; value (none) -> 1u
- C7: renamed from C?; value (none) -> 77u
- D1: renamed from D?; value (none) -> B230; footprint (none) -> Diode_SMD:D_SMB
- L1: renamed from L?; value (none) -> 10u
- Q1: renamed from Q?; value (none) -> CSD17553Q5A; footprint (none) -> Package_TO_SOT_SMD:TDSON-8-1
- R1: renamed from R?; value (none) -> 20
- R2: renamed from R?; value (none) -> 909
- R3: renamed from R?; value (none) -> 51.1k
- R4: renamed from R?; value (none) -> 100
- R5: renamed from R?; value (none) -> 25m
- R6: renamed from R?; value (none) -> 29.4k
- R7: renamed from R?; value (none) -> 10k
- SC1: renamed from SC?; value (none) -> Solar_Cell
- U1: renamed from U?; value (none) -> LM3478MA_NOPB; footprint (none) -> Texas_Instruments-LM3478MA_NOPB-*
Connections:
- net GND: now also BT1.2 (-), C1.2, C2.2, C3.2, C4.2, C5.2, C7.2, R3.2, R5.2, R7.2, SC1.2 (-), U1.4 (AGND), U1.5 (PGND)

Commit message: Final schematic and PCB created plus BOM and gerber files
Parts:
- removed BT1: Battery_Cell, symbol Device:Battery_Cell
- added J1: (no value), symbol Connector:USB_A
- C1, L1: value 10u -> (none)
- C2: value 100n -> (none)
- C3: value 82n -> (none)
- C4: value 195p -> (none)
- C5: value 1n -> (none)
- C6: value 1u -> (none)
- C7: value 77u -> (none)
- D1: value B230 -> (none); footprint Diode_SMD:D_SMB -> (none)
- Q1: footprint Package_TO_SOT_SMD:TDSON-8-1 -> (none)
- R1: value 20 -> (none)
- R2: value 909 -> (none)
- R3: value 51.1k -> (none)
- R4: value 100 -> (none)
- R5: value 25m -> (none)
- R6: value 29.4k -> (none)
- R7: value 10k -> (none)
- U1: value LM3478MA_NOPB -> (none); footprint Texas_Instruments-LM3478MA_NOPB-* -> (none)
Connections:
- net GND: now also J1.4 (GND), J1.5 (Shield)
- net at C7.1, D1.1 (K), R6.1: now also J1.1 (VBUS)
- no-connect marks 0 -> 2
