File: Schematics/SolarChargerV2/SolarChargerV2.kicad_pcb (KiCad board)
At the start: 2 copper layers, 73.7 x 40.6 mm, 20 parts, among them J1 USB_A, Q1 CSD17553Q5A, U1 LM3478MA_NOPB

Commit message: File rearangement and V3 of the project
Parts:
- removed Le: 10u, SolarChargelibrary:DRQ
- added L1: 10u, SolarChargelibrary:DRQ, F.Cu at (112.5, 60.2)
- C4: value 195p -> 200p
- C7: value 77u -> 47u
Routing:
- net Net-(C6-Pad1): track 37.6 -> 63.9 mm
- net Net-(C6-Pad2): track 25.4 -> 43.8 mm
- net Net-(C1-Pad1): track 30.2 -> 45.9 mm
- net GND: track 161.9 -> 169.0 mm
Changed lines of the file:
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@@
   )
   (footprint "SolarChargelibrary:DRQ" (layer "F.Cu")
-    (at 111.76 60.96 180)
+    (at 112.5 60.2)
     (property "Sheetfile" "SolarChargerV2.kicad_sch")
     (property "Sheetname" "")
     (attr through_hole)
-    (fp_text reference "Le" (at -8.4 0 90) (layer "F.SilkS")
+    (fp_text reference "L1" (at -8.4 0 90) (layer "F.SilkS")
       (effects (font (size 1 1) (thickness 0.15)))
     )
@@
     (fp_line (start -6.6 3.25) (end -7.4 2.45) (layer "F.SilkS") (width 0.12))
     (fp_line (start 7.4 -3.25) (end 7.4 3.25) (layer "F.SilkS") (width 0.12))
-    (fp_line (start -7.4 -3.25) (end 7.4 -3.25) (layer "F.SilkS") (width 0.12))
     (fp_line (start -7.4 2.45) (end -7.4 -3.25) (layer "F.SilkS") (width 0.12))
     (fp_line (start 7.4 3.25) (end -6.6 3.25) (layer "F.SilkS") (width 0.12))
+    (fp_line (start -7.4 -3.25) (end 7.4 -3.25) (layer "F.SilkS") (width 0.12))
     (fp_line (start -7.15 3) (end -7.15 -3) (layer "F.CrtYd") (width 0.05))
     (fp_line (start -7.15 -3) (end 7.15 -3) (layer "F.CrtYd") (width 0.05))
     (fp_line (start 7.15 -3) (end 7.15 3) (layer "F.CrtYd") (width 0.05))
     (fp_line (start 7.15 3) (end -7.15 3) (layer "F.CrtYd") (width 0.05))
-    (pad "1" smd rect (at -4.975 1.5 180) (size 3.85 2.5) (layers "F.Cu" "F.Paste" "F.Mask")
+    (pad "1" smd rect (at -4.975 1.5) (size 3.85 2.5) (layers "F.Cu" "F.Paste" "F.Mask")
       (net 12 "Net-(C6-Pad1)") (pinfunction "1") (pintype "passive"))
-    (pad "2" smd rect (at -4.975 -1.5 180) (size 3.85 2.5) (layers "F.Cu" "F.Paste" "F.Mask")
+    (pad "2" smd rect (at -4.975 -1.5) (size 3.85 2.5) (layers "F.Cu" "F.Paste" "F.Mask")
       (net 13 "Net-(C6-Pad2)") (pinfunction "2") (pintype "passive"))
-    (pad "3" smd rect (at 4.975 -1.5 180) (size 3.85 2.5) (layers "F.Cu" "F.Paste" "F.Mask")
+    (pad "3" smd rect (at 4.975 -1.5) (size 3.85 2.5) (layers "F.Cu" "F.Paste" "F.Mask")
       (net 5 "Net-(C1-Pad1)") (pinfunction "3") (pintype "passive"))
-    (pad "4" smd rect (at 4.975 1.5 180) (size 3.85 2.5) (layers "F.Cu" "F.Paste" "F.Mask")
+    (pad "4" smd rect (at 4.975 1.5) (size 3.85 2.5) (layers "F.Cu" "F.Paste" "F.Mask")
       (net 4 "GND") (pinfunction "4") (pintype "passive"))
   )
@@
       (effects (font (size 1 1) (thickness 0.15)))
     )
-    (fp_text value "77u" (at -5.715 0 180) (layer "F.Fab")
+    (fp_text value "47u" (at -5.715 0 180) (layer "F.Fab")
       (effects (font (size 1 1) (thickness 0.15)))
     )
@@
       (effects (font (size 1 1) (thickness 0.15)))
     )
-    (fp_text value "195p" (at 5.715 0 180) (layer "F.Fab")
+    (fp_text value "200p" (at 5.715 0 180) (layer "F.Fab")
       (effects (font (size 1 1) (thickness 0.15)))
     )
@@
   (segment (start 154.94 59.69) (end 154.83 59.8) (width 0.25) (layer "F.Cu") (net 4))
   (segment (start 109.855 79.375) (end 111.5325 79.375) (width 0.25) (layer "F.Cu") (net 4))
+  (segment (start 117.475 61.7) (end 116 61.7) (width 0.25) (layer "F.Cu") (net 4))
   (segment (start 137.16 83.88) (end 138.0125 83.88) (width 0.25) (layer "F.Cu") (net 4))
   (segment (start 152.12 67.62) (end 150.17 67.62) (width 0.25) (layer "F.Cu") (net 4))
@@
   (segment (start 111.76 83.185) (end 111.9925 83.4175) (width 0.25) (layer "F.Cu") (net 4))
   (segment (start 116.84 83.4175) (end 123.235 83.4175) (width 0.25) (layer "F.Cu") (net 4))
+  (segment (start 113.3 64.4) (end 101 64.4) (width 0.25) (layer "F.Cu") (net 4))
   (segment (start 109.625 82.78) (end 109.855 82.55) (width 0.25) (layer "F.Cu") (net 4))
-  (segment (start 101.195 59.46) (end 100.965 59.69) (width 0.25) (layer "F.Cu") (net 4))
   (segment (start 126.0375 83.77) (end 124.46 82.1925) (width 0.25) (layer "F.Cu") (net 4))
   (segment (start 129.54 83.77) (end 126.0375 83.77) (width 0.25) (layer "F.Cu") (net 4))
@@
   (segment (start 147.09 65) (end 147.32 64.77) (width 0.25) (layer "F.Cu") (net 4))
   (segment (start 111.76 74.5225) (end 110.2625 74.5225) (width 0.25) (layer "F.Cu") (net 4))
+  (segment (start 116 61.7) (end 113.3 64.4) (width 0.25) (layer "F.Cu") (net 4))
   (segment (start 124.525 74.23) (end 124.46 74.295) (width 0.25) (layer "F.Cu") (net 4))
-  (segment (start 106.785 59.46) (end 101.195 59.46) (width 0.25) (layer "F.Cu") (net 4))
+  (segment (start 101 64.4) (end 100.965 64.365) (width 0.25) (layer "F.Cu") (net 4))
   (segment (start 111.9925 83.4175) (end 116.84 83.4175) (width 0.25) (layer "F.Cu") (net 4))
   (segment (start 127 81.915) (end 124.7375 81.915) (width 0.25) (layer "F.Cu") (net 4))
@@
   (segment (start 147.32 59.69) (end 154.94 59.69) (width 0.25) (layer "F.Cu") (net 4))
   (via (at 127 81.915) (size 0.8) (drill 0.4) (layers "F.Cu" "B.Cu") (net 4))
+  (via (at 100.965 64.365) (size 0.8) (drill 0.4) (layers "F.Cu" "B.Cu") (net 4))
   (via (at 127 74.2055) (size 0.8) (drill 0.4) (layers "F.Cu" "B.Cu") (net 4))
   (via (at 147.32 64.77) (size 0.8) (drill 0.4) (layers "F.Cu" "B.Cu") (net 4))
-  (via (at 100.965 59.69) (size 0.8) (drill 0.4) (layers "F.Cu" "B.Cu") (net 4))
   (via (at 104.14 76.835) (size 0.8) (drill 0.4) (layers "F.Cu" "B.Cu") (net 4))
   (via (at 147.32 59.69) (size 0.8) (drill 0.4) (layers "F.Cu" "B.Cu") (net 4))
@@
   (via (at 109.855 82.55) (size 0.8) (drill 0.4) (layers "F.Cu" "B.Cu") (net 4))
   (segment (start 147.32 64.77) (end 147.32 59.69) (width 0.25) (layer "B.Cu") (net 4))
-  (segment (start 100.965 59.69) (end 100.965 73.66) (width 0.25) (layer "B.Cu") (net 4))
   (segment (start 104.14 83.82) (end 104.14 76.835) (width 0.25) (layer "B.Cu") (net 4))
   (segment (start 127 74.2055) (end 127 81.915) (width 0.25) (layer "B.Cu") (net 4))
   (segment (start 109.855 82.55) (end 109.855 79.375) (width 0.25) (layer "B.Cu") (net 4))
+  (segment (start 100.965 64.365) (end 100.965 73.66) (width 0.25) (layer "B.Cu") (net 4))
   (segment (start 109.855 74.93) (end 109.855 79.375) (width 0.25) (layer "B.Cu") (net 4))
   (segment (start 106.68 79.78) (end 107.545 79.78) (width 0.25) (layer "F.Cu") (net 5))
   (segment (start 108.8625 67.6675) (end 107.95 68.58) (width 0.25) (layer "F.Cu") (net 5))
+  (segment (start 104.975 63.7) (end 103.505 62.23) (width 0.25) (layer "F.Cu") (net 5))
+  (segment (start 113 58.7) (end 112.1 59.6) (width 0.25) (layer "F.Cu") (net 5))
   (segment (start 107.95 68.58) (end 104.14 68.58) (width 0.25) (layer "F.Cu") (net 5))
-  (segment (start 106.785 62.46) (end 103.735 62.46) (width 0.25) (layer "F.Cu") (net 5))
-  (segment (start 103.735 62.46) (end 103.505 62.23) (width 0.25) (layer "F.Cu") (net 5))
+  (segment (start 117.475 58.7) (end 113 58.7) (width 0.25) (layer "F.Cu") (net 5))
+  (segment (start 112.1 59.6) (end 112.1 63.7) (width 0.25) (layer "F.Cu") (net 5))
   (segment (start 111.76 67.6675) (end 108.8625 67.6675) (width 0.25) (layer "F.Cu") (net 5))
+  (segment (start 112.1 63.7) (end 104.975 63.7) (width 0.25) (layer "F.Cu") (net 5))
   (segment (start 107.545 79.78) (end 107.95 79.375) (width 0.25) (layer "F.Cu") (net 5))
   (via (at 103.505 62.23) (size 0.8) (drill 0.4) (layers "F.Cu" "B.Cu") (net 5))
@@
   (segment (start 133.985 71.755) (end 133.985 75.4755) (width 0.25) (layer "B.Cu") (net 11))
   (segment (start 137.16 70.07) (end 132.935 70.07) (width 0.25) (layer "F.Cu") (net 12))
-  (segment (start 116.735 59.46) (end 122.8625 59.46) (width 0.25) (layer "F.Cu") (net 12))
-  (segment (start 122.8625 59.46) (end 124.3625 60.96) (width 0.25) (layer "F.Cu") (net 12))
+  (segment (start 104.5 54.9) (end 122.5 54.9) (width 0.25) (layer "F.Cu") (net 12))
+  (segment (start 122.5 54.9) (end 124.3625 56.7625) (width 0.25) (layer "F.Cu") (net 12))
+  (segment (start 104.6 61.7) (end 104.5 61.6) (width 0.25) (layer "F.Cu") (net 12))
   (segment (start 124.46 57.15) (end 124.3625 57.2475) (width 0.25) (layer "F.Cu") (net 12))
   (segment (start 132.935 70.07) (end 132.715 69.85) (width 0.25) (layer "F.Cu") (net 12))
   (segment (start 124.3625 57.2475) (end 124.3625 60.96) (width 0.25) (layer "F.Cu") (net 12))
+  (segment (start 104.5 61.6) (end 104.5 54.9) (width 0.25) (layer "F.Cu") (net 12))
   (segment (start 132.715 57.15) (end 124.46 57.15) (width 0.25) (layer "F.Cu") (net 12))
+  (segment (start 124.3625 56.7625) (end 124.3625 60.96) (width 0.25) (layer "F.Cu") (net 12))
+  (segment (start 107.525 61.7) (end 104.6 61.7) (width 0.25) (layer "F.Cu") (net 12))
   (via (at 132.715 69.85) (size 0.8) (drill 0.4) (layers "F.Cu" "B.Cu") (net 12))
   (via (at 132.715 57.15) (size 0.8) (drill 0.4) (layers "F.Cu" "B.Cu") (net 12))
   (segment (start 132.715 69.85) (end 132.715 57.15) (width 0.25) (layer "B.Cu") (net 12))
+  (segment (start 107.525 56.025) (end 107.5 56) (width 0.25) (layer "F.Cu") (net 13))
   (segment (start 135.01 60.96) (end 129.6375 60.96) (width 0.25) (layer "F.Cu") (net 13))
+  (segment (start 107.525 58.7) (end 107.525 56.025) (width 0.25) (layer "F.Cu") (net 13))
   (segment (start 121.285 65.405) (end 129.54 65.405) (width 0.25) (layer "F.Cu") (net 13))
-  (segment (start 116.735 62.46) (end 120.88 62.46) (width 0.25) (layer "F.Cu") (net 13))
   (segment (start 129.6375 65.3075) (end 129.6375 60.96) (width 0.25) (layer "F.Cu") (net 13))
-  (segment (start 120.88 62.46) (end 121.285 62.865) (width 0.25) (layer "F.Cu") (net 13))
+  (segment (start 121.285 56.385) (end 121.285 62.865) (width 0.25) (layer "F.Cu") (net 13))
+  (segment (start 107.5 56) (end 120.9 56) (width 0.25) (layer "F.Cu") (net 13))
+  (segment (start 120.9 56) (end 121.285 56.385) (width 0.25) (layer "F.Cu") (net 13))
   (segment (start 129.54 65.405) (end 129.6375 65.3075) (width 0.25) (layer "F.Cu") (net 13))
   (via (at 121.285 65.405) (size 0.8) (drill 0.4) (layers "F.Cu" "B.Cu") (net 13))
