File: Schematics/SolarChargerV2/SolarChargerV2.kicad_pcb (KiCad board)
At the start: 2 copper layers, 73.7 x 40.6 mm, 20 parts, among them J1 USB_A, Q1 CSD16410Q5A, U1 LM3478MA_NOPB

Commit message: changes
Parts:
- C1: footprint Capacitor_SMD:CP_Elec_3x5.3 -> Capacitor_SMD:C_1812_4532Metric
- C2, C3, C5: footprint Capacitor_SMD:C_0603_1608Metric_Pad1.08x0.95mm_HandSolder -> Capacitor_SMD:C_0402_1005Metric
- C4: footprint Capacitor_SMD:C_1812_4532Metric_Pad1.57x3.40mm_HandSolder -> Capacitor_SMD:C_0603_1608Metric
- C6: footprint Capacitor_SMD:C_2220_5650Metric_Pad1.97x5.40mm_HandSolder -> Capacitor_SMD:C_0805_2012Metric
- C7: footprint Capacitor_SMD:CP_Elec_3x5.3 -> Capacitor_SMD:C_1206_3216Metric
- R1, R3, R4: footprint Resistor_SMD:R_0603_1608Metric_Pad0.98x0.95mm_HandSolder -> Resistor_SMD:R_0603_1608Metric
- R2, R5: footprint Resistor_SMD:R_2816_7142Metric_Pad3.20x4.45mm_HandSolder -> Resistor_SMD:R_1206_3216Metric
- R6: footprint Resistor_SMD:R_0603_1608Metric_Pad0.98x0.95mm_HandSolder -> Resistor_SMD:R_0402_1005Metric
- moved L1 6.37 mm to (107.9, 55.8)
- moved SC1 4.04 mm to (100.7, 69.0)
Routing:
- net Net-(C6-Pad2): track 43.8 -> 56.7 mm, vias 2 -> 4
- net GND: track 169.0 -> 177.7 mm
- net Net-(Q1-Pad5): track 63.9 -> 70.5 mm, vias 2 -> 6
- net Net-(C4-Pad1): track 20.7 -> 23.2 mm
- net Net-(C3-Pad1): track 9.00 -> 10.1 mm
- net Net-(C5-Pad1): track 27.7 -> 28.8 mm
- net Net-(C1-Pad1): track 45.9 -> 45.4 mm, vias 3 -> 4
Other:
- board size 73.7 x 40.6 mm -> 74.5 x 47.6 mm
