File: Schematics/SolarChargerV2/SolarChargerV2.kicad_sch (KiCad schematic)
At the start: 20 parts, among them Q1 CSD17553Q5A

Commit message: File rearangement and V3 of the project
Parts:
- C1: value (none) -> 10u; footprint (none) -> Capacitor_SMD:CP_Elec_3x5.3
- C2: value (none) -> 100n; footprint (none) -> Capacitor_SMD:C_0603_1608Metric_Pad1.08x0.95mm_HandSolder
- C3: value (none) -> 82n; footprint (none) -> Capacitor_SMD:C_0603_1608Metric_Pad1.08x0.95mm_HandSolder
- C4: footprint (none) -> Capacitor_SMD:C_1812_4532Metric_Pad1.57x3.40mm_HandSolder
- C5: value (none) -> 1n; footprint (none) -> Capacitor_SMD:C_0603_1608Metric_Pad1.08x0.95mm_HandSolder
- C6: value (none) -> 1u; footprint (none) -> Capacitor_SMD:C_2220_5650Metric_Pad1.97x5.40mm_HandSolder
- C7: footprint (none) -> Capacitor_SMD:CP_Elec_3x5.3
- D1: value (none) -> B230; footprint (none) -> Diode_SMD:D_SMB
- J1: value (none) -> USB_A; footprint (none) -> Connector_USB:USB_A_Molex_67643_Horizontal
- L1: value (none) -> 10u; footprint (none) -> SolarChargelibrary:DRQ
- Q1: footprint (none) -> Package_TO_SOT_SMD:TDSON-8-1
- R1: value (none) -> 20; footprint (none) -> Resistor_SMD:R_0603_1608Metric_Pad0.98x0.95mm_HandSolder
- R2: value (none) -> 909; footprint (none) -> Resistor_SMD:R_2816_7142Metric_Pad3.20x4.45mm_HandSolder
- R3: value (none) -> 51.1k; footprint (none) -> Resistor_SMD:R_0603_1608Metric_Pad0.98x0.95mm_HandSolder
- R4: value (none) -> 100; footprint (none) -> Resistor_SMD:R_0603_1608Metric_Pad0.98x0.95mm_HandSolder
- R5: value (none) -> 25m; footprint (none) -> Resistor_SMD:R_2816_7142Metric_Pad3.20x4.45mm_HandSolder
- R6: value (none) -> 29.4k; footprint (none) -> Resistor_SMD:R_0603_1608Metric_Pad0.98x0.95mm_HandSolder
- R7: value (none) -> 10k; footprint (none) -> Resistor_SMD:R_0805_2012Metric
- SC1: footprint (none) -> SolarChargelibrary:SIP-2
- U1: value (none) -> LM3478MA_NOPB; footprint (none) -> Package_SO:SOIC-8_3.9x4.9mm_P1.27mm
