File: Schematics/SolarChargerV2/SolarChargerV2.kicad_sch (KiCad schematic)
At the start: 20 parts, among them J1 USB_A, U1 LM3478MA_NOPB

Commit message: changes
Parts:
- C1: value 10u -> (none); footprint Capacitor_SMD:CP_Elec_3x5.3 -> (none)
- C2: value 100n -> (none); footprint Capacitor_SMD:C_0603_1608Metric_Pad1.08x0.95mm_HandSolder -> (none)
- C3: value 82n -> (none); footprint Capacitor_SMD:C_0603_1608Metric_Pad1.08x0.95mm_HandSolder -> (none)
- C4: value 200p -> (none); footprint Capacitor_SMD:C_1812_4532Metric_Pad1.57x3.40mm_HandSolder -> (none)
- C5: value 1n -> (none); footprint Capacitor_SMD:C_0603_1608Metric_Pad1.08x0.95mm_HandSolder -> (none)
- C6: value 1u -> (none); footprint Capacitor_SMD:C_2220_5650Metric_Pad1.97x5.40mm_HandSolder -> (none)
- C7: value 47u -> (none); footprint Capacitor_SMD:CP_Elec_3x5.3 -> (none)
- R1: value 20 -> (none); footprint Resistor_SMD:R_0603_1608Metric_Pad0.98x0.95mm_HandSolder -> (none)
- R3: value 51.1k -> (none); footprint Resistor_SMD:R_0603_1608Metric_Pad0.98x0.95mm_HandSolder -> (none)
- R4: value 100 -> (none); footprint Resistor_SMD:R_0603_1608Metric_Pad0.98x0.95mm_HandSolder -> (none)
- R5: value 25m -> (none); footprint Resistor_SMD:R_2816_7142Metric_Pad3.20x4.45mm_HandSolder -> (none)
- R6: value 29.4k -> (none); footprint Resistor_SMD:R_0603_1608Metric_Pad0.98x0.95mm_HandSolder -> (none)
- R7: value 10k -> (none); footprint Resistor_SMD:R_0805_2012Metric -> (none)
