File: Schematics/SolarChargerV6/SolarChargerV6.kicad_sch (KiCad schematic)
At the start: 20 parts, among them J1 USB_A, Q1 CSD16410Q5A, U1 LM3478MA_NOPB

Commit message: Updates
Parts:
- added R10, R11, R8, R9: (no value), symbol Device:R
- C1: value (none) -> 10u; footprint (none) -> Capacitor_SMD:C_1812_4532Metric
- C2: value (none) -> 100n; footprint (none) -> Capacitor_SMD:C_0805_2012Metric
- C3: value (none) -> 82n; footprint (none) -> Capacitor_SMD:C_0603_1608Metric
- C4: value (none) -> 200p; footprint (none) -> Capacitor_SMD:C_0805_2012Metric
- C5: value (none) -> 1n; footprint (none) -> Capacitor_SMD:C_0805_2012Metric
- C6: value (none) -> 1u; footprint (none) -> Capacitor_SMD:C_0805_2012Metric
- C7: value (none) -> 47u; footprint (none) -> Capacitor_SMD:C_1206_3216Metric
- R1: value (none) -> 20; footprint (none) -> Resistor_SMD:R_0603_1608Metric
- R2: value (none) -> 887; footprint (none) -> Resistor_SMD:R_1206_3216Metric
- R3: value (none) -> 51.1k; footprint (none) -> Resistor_SMD:R_0805_2012Metric
- R4: value (none) -> 100; footprint (none) -> Resistor_SMD:R_0805_2012Metric
- R5: value (none) -> 25m; footprint (none) -> Resistor_SMD:R_1206_3216Metric
- R6: value (none) -> 29.4k; footprint (none) -> Resistor_SMD:R_0805_2012Metric
- R7: value (none) -> 10k; footprint (none) -> Resistor_SMD:R_0805_2012Metric
Connections:
- net GND: now also R11.2, R9.2
- net at C7.1, D1.1 (K), J1.1 (VBUS)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: now also R10.1, R8.1
- net at J1.2 (D-): now also R10.2, R11.1
- net at J1.3 (D+): now also R8.2, R9.1
- no-connect marks 2 -> 0
Other:
- moved on the sheet: C1, C2, C3, C4, C5, C6, C7, D1, J1, L1, Q1, R1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
